File: TempBoost.sch (KiCad schematic (older format))
At the start: 28 parts, among them J1 Conn_01x02, J2 Conn_01x02, Q201 Q_NMOS_GSD, T1 Transformer_1P_1S, U201 MIC2920

Commit message: Added OPAx140 Library and added compensator network
Parts:
- removed C207, C209: 2.2nF, Capacitors_SMD:C_0805, symbol C
- removed C208: 4.7nF, Capacitors_SMD:C_0805, symbol C
- removed R201: 118K, symbol R
- removed R202: 13.7k, symbol R
- removed R203: 453k, symbol R
- removed R204: 2M, symbol R
- added C207, C209: 2.2uF, symbol C_Small
- added C208: 4.7nF, symbol C_Small
- added C?: C, symbol C
- added R201: 118K, symbol R_Small
- added R202: 13.7K, symbol R_Small
- added R203: 562, symbol R_Small
- added R204: 1M, symbol R_Small
- added R?: R, symbol R
- added U?: OPA140, symbol OPA140
Connections:
- net labels added: +12V, LOAD+, LOAD-, VFB, VRECT+, VRECT-, VREF
- wire segments 36 -> 66
Other:
- note added: "120VAC -> 25VDC Rectifier"
- note added: "Amplifier Bias Supply"
- note added: "Error Amp"
- note added: "Why two connectors?"
- moved on the sheet: C201, C202, C203, C204, C205, C206, C210, C211, C212, D1, D2, D202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

Commit message: Added Components
Parts:
- added C213, C215: 1uF, Capacitors_SMD:C_0805, symbol C
- added C214: 100nF, Capacitors_SMD:C_0603, symbol C
- added R205, R206: 10k, Resistors_SMD:R_0805, symbol R
- added U203: UCC27517A, symbol UCC27517A
- added U204: AD1582, TO_SOT_Packages_SMD:SOT-23, symbol AD1582
- added U205: LM2904, Housings_SOIC:SOIC-8_3.9x4.9mm_Pitch1.27mm, symbol LM2904
- gave numbers to parts that had none: 1
- renumbered D202 to D201
Connections:
- net labels added: Gate, VPMM
- wire segments 66 -> 120
Other:
- note added: "2.5V Reference"
- note added: "Gate Drier"

Commit message: Added Triangle Generator
Parts:
- removed U202: OPA140, symbol OPA140
- added C? (x2): 1uF, Capacitors_SMD:C_0805, symbol C
- added R? (x3): 10k, Resistors_SMD:R_0805, symbol R
- added RV1: POT, symbol POT
- added U202: OPA2140, Housings_SOIC:SOIC-8_3.9x4.9mm_Pitch1.27mm, symbol OPA2140
Connections:
- net labels added: VPWM, VTRI
- net labels removed: LOAD-, VPMM
- wire segments 120 -> 95
Other:
- note added: "Triangle Wave Generator"
- note removed: "Why two connectors?"
- moved on the sheet: C207, C208, C209, C213, C214, C215, R201, R202, R203, R204, R206, U205A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

Commit message: Load Switch
Parts:
- removed R?: R, symbol R
- added U206: TPS1H100, symbol TPS1H100
- C201, C202: symbol C -> CP
- C207: value 2.2uF -> 6800pF
- C208: value 4.7nF -> 7500pF
- C209: value 2.2uF -> 1pF
- R203: value 562 -> 130k
- R204: value 1M -> 3k
Connections:
- wire segments 95 -> 111
- no-connect marks 0 -> 3
Other:
- moved on the sheet: C203, C204, C205, C206, C?, D201, L1, Q201, R?, RV1, U202B, U203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

Commit message: Transformer
Parts:
- removed C?: C, symbol C
- removed D1, D2, D3, D4: D, symbol D
- removed F1: Fuse, symbol Fuse
- removed J1: Conn_01x02, symbol Conn_01x02
- removed T1: Transformer_1P_1S, symbol Transformer_1P_1S
- added C101, C102: 2200uF, symbol CP
- added C103, C104: 220uF, symbol CP
- added F?: Fuse, symbol Fuse
- added J?: Conn_01x02, symbol Conn_01x02
- added RV2: 5k, symbol POT
- added SW?: SW_SPST, symbol SW_SPST
- added T?: 3FD-224, symbol 3FD-224
- added U?: DF005S2, symbol DF005S2
- R202: value 13.7K -> 10K
Connections:
- wire segments 111 -> 119
Other:
- note removed: "120VAC -> 25VDC Rectifier"

Commit message: fixed voltage reference
Parts:
- U204: value AD1582 -> 2925; symbol AD1582 -> 2925; Manufactuer Analog Devices -> Texas Instruments; Part Number AD1582WBRTZ-R7 -> REF2925AIDBZR
- gave numbers to parts that had none: 2
Connections:
- wire segments 119 -> 178
Other:
- moved on the sheet: C201, C202, C203, C204, C205, C206, D201, L1, Q201, U204, U206

Commit message: Update
Parts:
- RV1: value POT -> 5k
Connections:
- net labels added: VSWITCHED
- wire segments 178 -> 125
Other:
- moved on the sheet: U206
Changed lines of the file:
@@
 $EndComp
 Text GLabel 1107 3851 0    39   Input ~ 0
-VRECT+
+VSWITCHED
 Text GLabel 1117 4501 0    39   Input ~ 0
 VRECT-
@@
 VRECT-
 Wire Wire Line
-	3150 6100 3300 6100
-Wire Wire Line
-	3300 6100 3700 6100
+	3150 6100 3700 6100
 Connection ~ 3300 6100
 Connection ~ 2400 6100
@@
 	1107 3851 1367 3851
 Wire Wire Line
-	2120 6100 2400 6100
-Wire Wire Line
-	2400 6100 2550 6100
+	2120 6100 2550 6100
 Connection ~ 3700 6100
-Text GLabel 5800 3850 2    39   Input ~ 0
+Text GLabel 4600 3850 2    39   Input ~ 0
 LOAD+
 Text Notes 2535 5715 0    39   ~ 0
@@
 	8385 1475 8245 1475
 Wire Wire Line
-	8245 2035 8245 1475
-Wire Wire Line
-	8245 1475 8245 1195
+	8245 2035 8245 1195
 Wire Wire Line
 	8245 1195 8665 1195
@@
 	8865 1195 9590 1195
 Wire Wire Line
-	9590 1195 9590 1475
-Wire Wire Line
-	9590 1475 9590 2135
+	9590 1195 9590 2135
 Wire Wire Line
 	9590 1475 9180 1475
 Wire Wire Line
-	7175 2035 7450 2035
-Wire Wire Line
-	7450 2035 7705 2035
-Wire Wire Line
-	7705 2035 8245 2035
-Wire Wire Line
-	8245 2035 8555 2035
+	7175 2035 8555 2035
 Connection ~ 8245 1475
 Wire Wire Line
-	9505 2135 9590 2135
-Wire Wire Line
-	9590 2135 9750 2135
+	9505 2135 9750 2135
 Connection ~ 9590 1475
 Text GLabel 9750 2135 2    39   Input ~ 0
@@
 Connection ~ 7450 2035
 Wire Wire Line
-	6575 2035 6710 2035
-Wire Wire Line
-	6710 2035 6975 2035
+	6575 2035 6975 2035
 Wire Wire Line
 	6710 2035 6710 2195
@@
 	6100 7250 6100 6950
 Wire Wire Line
-	4800 7250 4950 7250
-Wire Wire Line
-	4950 7250 6100 7250
+	4800 7250 6100 7250
 Wire Wire Line
 	4950 7250 4950 6850
@@
 	2400 6445 2400 6495
 Wire Wire Line
-	3300 6095 3300 6100
-Wire Wire Line
-	3300 6100 3300 6135
+	3300 6095 3300 6135
 Wire Wire Line
 	2400 6145 2400 6100
 Wire Wire Line
-	2125 6495 2400 6495
-Wire Wire Line
-	2400 6495 3300 6495
-Wire Wire Line
-	3300 6495 3700 6495
+	2125 6495 3700 6495
 Connection ~ 2400 6495
 Connection ~ 3300 6495
@@
 	3300 6495 3300 6435
 Wire Wire Line
-	3700 6070 3700 6100
-Wire Wire Line
-	3700 6100 3700 6135
+	3700 6070 3700 6135
 $Comp
 L +12V #PWR05
@@
 $EndComp
 Wire Wire Line
-	8500 3300 8750 3300
-Wire Wire Line
-	8750 3300 9100 3300
-Wire Wire Line
-	9100 3300 9350 3300
+	8400 3300 9350 3300
 Connection ~ 8750 3300
 Connection ~ 9100 3300
 Wire Wire Line
-	6950 3700 8050 3700
-Wire Wire Line
-	8050 3700 8500 3700
-Wire Wire Line
-	8500 3700 8750 3700
-Wire Wire Line
-	8750 3700 9100 3700
-Wire Wire Line
-	8500 3300 8500 3300
-Wire Wire Line
-	8500 3300 8500 3700
+	6950 3700 9100 3700
 Connection ~ 8750 3700
 Wire Wire Line
-	6950 3300 7400 3300
-Wire Wire Line
-	7400 3300 7700 3300
+	6950 3300 7700 3300
 Connection ~ 7400 3300
-Connection ~ 8500 3700
 Connection ~ 8050 3700
 Text Notes 5300 6300 0    39   ~ 0
@@
 VFB
 Wire Wire Line
-	9250 5750 9300 5750
-Wire Wire Line
-	9300 5750 9750 5750
+	9250 5750 9750 5750
 Text Label 9400 5750 0    39   ~ 0
 VTRI
@@
 P 6650 5300
 F 0 "RV1" V 6475 5300 50  0000 C CNN
-F 1 "POT" V 6550 5300 50  0000 C CNN
+F 1 "5k" V 6550 5300 50  0000 C CNN
 F 2 "" H 6650 5300 50  0001 C CNN
 F 3 "" H 6650 5300 50  0001 C CNN
@@
 	6800 5300 6800 5150
 Wire Wire Line
-	6650 5150 6800 5150
-Wire Wire Line
-	6800 5150 7750 5150
+	6650 5150 7750 5150
 Wire Wire Line
 	7750 5150 7750 5850
@@
 	7750 5850 7900 5850
 Wire Wire Line
-	8200 4850 8200 5150
-Wire Wire Line
-	8200 5150 8200 5850
+	8200 4850 8200 5850
 Wire Wire Line
 	8200 5850 8650 5850
@@
 $EndComp
 Wire Wire Line
-	9300 4850 9300 5150
-Wire Wire Line
-	9300 5150 9300 5750
+	9300 4850 9300 5750
 Wire Wire Line
 	9300 5150 9050 5150
@@
 L TPS1H100 U206
 U 1 1 5CA67357
-P 5050 3750
-F 0 "U206" H 5100 3250 60  0000 C CNN
-F 1 "TPS1H100" H 5050 4200 60  0000 C CNN
-F 2 "" H 5100 3800 60  0001 C CNN
-F 3 "" H 5100 3800 60  0001 C CNN
-	1    5050 3750
-	-1   0    0    -1
-$EndComp
-Wire Wire Line
-	5550 3850 5650 3850
-Wire Wire Line
-	5650 3850 5800 3850
-Wire Wire Line
-	5550 3950 5650 3950
-Wire Wire Line
-	5650 3850 5650 3950
-Wire Wire Line
-	5650 3950 5650 4050
-Connection ~ 5650 3850
-Wire Wire Line
-	5650 4050 5550 4050
-Connection ~ 5650 3950
-Wire Wire Line
-	4400 4050 4500 4050
-Wire Wire Line
-	4400 3850 4400 3950
-Wire Wire Line
-	4400 3950 4400 4050
-Wire Wire Line
-	2300 3850 2500 3850
-Wire Wire Line
-	2500 3850 2800 3850
-Wire Wire Line
-	2800 3850 3100 3850
-Wire Wire Line
-	3100 3850 3400 3850
-Wire Wire Line
-	3400 3850 3700 3850
-Wire Wire Line
-	3700 3850 4000 3850
-Wire Wire Line
-	4000 3850 4400 3850
-Wire Wire Line
-	4400 3850 4500 3850
-Wire Wire Line
-	4500 3950 4400 3950
-Connection ~ 4400 3950
-Connection ~ 4400 3850
+P 4800 2300
+F 0 "U206" H 4850 1800 60  0000 C CNN
+F 1 "TPS1H100" H 4800 2750 60  0000 C CNN
+F 2 "" H 4850 2350 60  0001 C CNN
+F 3 "" H 4850 2350 60  0001 C CNN
+	1    4800 2300
+	-1   0    0    -1
+$EndComp
+Wire Wire Line
+	5300 2400 5550 2400
+Wire Wire Line
+	5300 2500 5400 2500
+Wire Wire Line
+	5400 2400 5400 2600
+Connection ~ 5400 2400
+Wire Wire Line
+	5400 2600 5300 2600
+Connection ~ 5400 2500
+Wire Wire Line
+	4150 2600 4250 2600
+Wire Wire Line
+	4150 2400 4150 2600
+Wire Wire Line
+	2300 3850 4600 3850
+Wire Wire Line
+	3750 2400 4250 2400
+Wire Wire Line
+	4250 2500 4150 2500
+Connection ~ 4150 2500
+Connection ~ 4150 2400
 Connection ~ 2299 3851
 Wire Wire Line
-	4000 3950 4000 3850
+	4000 3850 4000 3950
 Connection ~ 4000 3850
 Wire Wire Line
@@
 	2500 4250 2500 4500
 Wire Wire Line
-	1200 4500 2500 4500
-Wire Wire Line
-	2500 4500 2800 4500
-Wire Wire Line
-	2800 4500 3100 4500
-Wire Wire Line
-	3100 4500 3400 4500
-Wire Wire Line
-	3400 4500 3700 4500
-Wire Wire Line
-	3700 4500 4000 4500
+	1200 4500 4000 4500
 Wire Wire Line
 	2800 4500 2800 4250
@@
 	2000 3850 2000 3849
 Wire Wire Line
-	1667 3850 1767 3850
-Wire Wire Line
-	1767 3850 2000 3850
+	1667 3850 2000 3850
 Connection ~ 2000 3851
 Connection ~ 1666 3849
@@
 Connection ~ 1767 3953
 Wire Wire Line
-	1395 4151 1396 4151
-Wire Wire Line
-	1396 4151 1467 4151
+	1395 4151 1467 4151
 Wire Wire Line
 	1395 4151 1395 4150
@@
 Wire Wire Line
 	1200 4501 1200 4500
-NoConn ~ 5550 3750
-NoConn ~ 5550 3450
-NoConn ~ 4500 3750
+NoConn ~ 5300 2300
+NoConn ~ 5300 2000
+NoConn ~ 4250 2300
 $Comp
 L POT RV2
@@
 	2050 1100 2100 1100
 Wire Wire Line
-	2400 1100 2500 1100
-Wire Wire Line
-	2500 1100 2600 1100
+	2400 1100 2600 1100
 Wire Wire Line
 	1400 1200 1650 1200
@@
 	1650 1200 1650 1500
 Wire Wire Line
-	1650 1500 2450 1500
-Wire Wire Line
-	2450 1500 2600 1500
+	1650 1500 2600 1500
 $Comp
 L CP C101
@@
 $EndComp
 Wire Wire Line
-	4350 1100 4900 1100
-Wire Wire Line
-	4900 1100 5300 1100
-Wire Wire Line
-	5300 1100 5750 1100
-Wire Wire Line
-	5750 1100 6200 1100
-Wire Wire Line
-	6200 1100 6650 1100
+	4350 1100 6650 1100
 $Comp
 L 3FD-224 T101
@@
 	3400 1500 3550 1500
 Wire Wire Line
-	4350 1500 4900 1500
-Wire Wire Line
-	4900 1500 5300 1500
-Wire Wire Line
-	5300 1500 5750 1500
-Wire Wire Line
-	5750 1500 6200 1500
-Wire Wire Line
-	6200 1500 6650 1500
+	4350 1500 6650 1500
 Wire Wire Line
 	4900 1500 4900 1450
@@
 VRECT-
 Connection ~ 6200 1500
-Connection ~ 8500 3300
 Wire Wire Line
 	8050 3550 8050 3700
@@
 	1    0    0    -1
 $EndComp
-Wire Wire Line
-	8400 3300 8500 3300
+Text GLabel 3750 2400 0    39   Input ~ 0
+VRECT+
+Text GLabel 5550 2400 2    39   Input ~ 0
+VSWITCHED
 $EndSCHEMATC

Commit message: Changed Triangle Wave
Parts:
- removed C214: 100nF, Capacitors_SMD:C_0603, symbol C
- removed C? (x2): 1uF, Capacitors_SMD:C_0805, symbol C
- removed R? (x3): 10k, Resistors_SMD:R_0805, symbol R
- removed RV1: 5k, symbol POT
- removed U202: OPA2140, Housings_SOIC:SOIC-8_3.9x4.9mm_Pitch1.27mm, symbol OPA2140
- added C? (x2): 1uF, Capacitors_SMD:C_0805, symbol C
- added D101, D204, D205: D_TVS, symbol D_TVS
- added R207: 60k, Resistors_SMD:R_0805, symbol R
- added R208: 10k, Resistors_SMD:R_0805, symbol R
- added RV2: POT, symbol POT
- added U205: LM1117-5.0, symbol LM1117-5.0
- gave numbers to parts that had none: 3
Connections:
- net labels added: +5V, OVSD
- net labels removed: VTRI
- wire segments 125 -> 133
Other:
- note added: "12V Supply"
- note added: "Output Overvoltage Trigger"
- note added: "Short circuit, overcurrent, undervoltage, reverse voltage Shutdown"
- note removed: "Amplifier Bias Supply"
- note removed: "Triangle Wave Generator"
- note removed: "Why 6 Capacitors?\n-> 220uF is the design total capacitance for this design.\nCapacitor ESR is a function of freqency, with smaller values\nand smaller packages having lower ESR at higher frequency.\nBy having a ground plane 'cage' with bypass capacitors\nspread over a larger range, generally by decade, you can provide a\nlow ESR path for low frequency transient response and high\nfrequency switc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"
- moved on the sheet: C210, C211, C212, C213, C215, J2, R205, R206, U201, U203, U204, U205A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
